File: 00-produccion-pcbs/1-versiones-profes/grupo-04/g-04-osc-02-rev-a/g-04-osc-02-rev-a.kicad_pcb (KiCad board)
At the start: 2 copper layers, 100 x 80 mm, 24 parts, among them J1 Barrel_Jack_Switch, J3 Barrel_Jack_Switch, J4 AudioJack2_SwitchT, J5 Conn_01x03_Pin, SW3 SW_SPDT, U1 40106, U5 L7805

Commit message: añadidoa g04-02
Parts:
- added R2: 1k, Resistor_THT:R_Axial_DIN0207_L6.3mm_D2.5mm_P10.16mm_Horizontal, F.Cu at (88.1, 69.8)
- D1: value D_Small -> 1n4148
- RVAR1, RVAR2: value 100K -> 100k
Connections:
- J4 pad 1: unconnected-(J4-Pad1) -> GND
- J4 pad 3: unconnected-(J4-Pad3) -> Output
- RVAR1 pad 1: Net-(D1-A) -> Net-(C1-Pad1)
- RVAR1 pad 2: Net-(C1-Pad1) -> Net-(D1-A)
- RVAR1 pad 3: (no net) -> unconnected-(RVAR1-Pad3)
- RVAR2 pad 1: Output -> Net-(C2-Pad1)
- RVAR2 pad 2: Net-(C2-Pad1) -> Net-(R2-Pad2)
- RVAR2 pad 3: (no net) -> unconnected-(RVAR2-Pad3)
- U1 pad 2: Output -> Net-(R2-Pad2)
Routing:
- net Net-(R2-Pad2): track 0.00 -> 86.1 mm, vias 0 -> 2
- net GND: track 0.00 -> 64.1 mm, vias 0 -> 3
- net +5V: track 83.0 -> 120.8 mm, vias 0 -> 2
- net Output: track 48.4 -> 33.3 mm
- net Net-(C2-Pad1): track 105.3 -> 117.0 mm
- net Net-(D1-A): track 60.2 -> 58.1 mm
- net Net-(C1-Pad1): track 66.7 -> 68.8 mm
- net +12V: track 133.0 -> 134.9 mm
Other:
- board text added: "g-04-osc-02-rev-a"
