File: 00-produccion-pcbs/1-versiones-profes/grupo-04/g-04-osc-02-rev-a/g-04-osc-02-rev-a.kicad_sch (KiCad schematic)
At the start: 31 parts, among them J1 Barrel_Jack_Switch, J3 Barrel_Jack_Switch, J4 AudioJack2_SwitchT, J5 Conn_01x03_Pin, SW3 SW_SPDT, U1 40106, U4 LM386, U5 L7805

Commit message: añadidoa g04-02
Parts:
- removed C10, C8, C9: 10u, Capacitor_THT:CP_Radial_D4.0mm_P2.00mm, symbol Device:C_Polarized
- removed C7: 100n, Capacitor_THT:C_Disc_D5.0mm_W2.5mm_P2.50mm, symbol Device:C
- removed LS1: Speaker, Connector_PinHeader_2.54mm:PinHeader_1x02_P2.54mm_Vertical, symbol Device:Speaker
- removed RV3: 100K, Potentiometer_THT:Potentiometer_Alps_RK163_Single_Horizontal, symbol Device:R_Potentiometer
- removed RVAR1, RVAR2: 100K, Potentiometer_THT:Potentiometer_Alps_RK163_Single_Horizontal, symbol Device:R_Variable
- removed U4: LM386, Package_DIP:DIP-8_W7.62mm, symbol Amplifier_Audio:LM386
- added R2: 1k, Resistor_THT:R_Axial_DIN0207_L6.3mm_D2.5mm_P10.16mm_Horizontal, symbol Device:R
- added RVAR1, RVAR2: 100k, Potentiometer_THT:Potentiometer_Alps_RK163_Single_Horizontal, symbol Device:R_Potentiometer
- D1: value D_Small -> 1n4148
Connections:
- net GND: now also J4.1
- net Output: now also J4.3, R2.1; no longer U1.2
- net at D1.2 (A), U1.12: now also RVAR1.2
- net at C1.1, U1.13: now also RVAR1.1
- net at C2.1, R1.1, U1.1: now also RVAR2.1
- new net: R2.2, RVAR2.2, U1.2
- no-connect marks 9 -> 10
Other:
- note removed: "cambiar numero de pines a este orden (reemplazar T/TN/S)"
- moved on the sheet: J4
